File: hardware/VFD_IV6.kicad_sch (KiCad schematic)
At the start: 95 parts, among them J1 Conn_01x10, Q2 BC817, U1 4511, U10 TBD62783A, U11 4511, U12 TBD62783A, U13 4017, U14 74HC04, U2 TBD62783A, U3 4511, U4 TBD62783A, U5 4511, U6 TBD62783A, U7 4511, U8 TBD62783A, U9 4511

Commit message: Updated schematic
Parts:
- removed C1: 100u, Capacitor_Tantalum_SMD:CP_EIA-7343-31_Kemet-D, symbol Device:C_Polarized_Small
- removed J1: Conn_01x10, Connector_PinHeader_2.54mm:PinHeader_1x09_P2.54mm_Vertical, symbol Connector_Generic:Conn_01x09
- removed R11, R12, R13, R14, R15, R16, R17, R2, R20, R21, R22, R23, R24, R25, R26, R29, R3, R30, R31, R32, R33, R34, R35, R38, R39, R4, R40, R41, R42, R43, R44, R47, R48, R49, R5, R50, R51, R52, R53, R6, R7, R8: 47k, Resistor_SMD:R_0603_1608Metric, symbol Device:R_Small
- removed U13: 4017, Package_DIP:DIP-16_W8.89mm_SMDSocket_LongPads, symbol 4xxx:4017
- removed VFD_PWR1: (no value), Library:VFD_PowerSupply, symbol CustomLibrary:VFD_PowerSupply
- added BT1: CR1220, Library:RSPRO1220, symbol Device:Battery_Cell
- added BZ1: Buzzer, Buzzer_Beeper:Buzzer_12x9.5RM7.6, symbol Device:Buzzer
- added C1, C10, C11, C12, C13, C14, C15, C21, C9: 100n, Capacitor_SMD:C_0603_1608Metric, symbol Device:C_Small
- added C16, C17: 22p, Capacitor_SMD:C_0603_1608Metric, symbol Device:C_Small
- added C18, C25: 10n, Capacitor_SMD:C_0603_1608Metric, symbol Device:C_Small
- added C19: 2u2, Capacitor_SMD:C_0805_2012Metric, symbol Device:C_Small
- added C20: 1u, Capacitor_SMD:C_0805_2012Metric, symbol Device:C_Small
- added C22: 3n9, Capacitor_SMD:C_0603_1608Metric, symbol Device:C_Small
- added C23, C24: 10u 25v, Capacitor_SMD:C_0805_2012Metric, symbol Device:C_Small
- added C26: 22u 6,3v, Capacitor_SMD:C_1210_3225Metric, symbol Device:C_Small
- added C27: 82p, Capacitor_SMD:C_0603_1608Metric, symbol Device:C_Small
- added C28: 10u, Capacitor_SMD:C_0805_2012Metric, symbol Device:C_Small
- added C29: 2u2 50v, Capacitor_SMD:C_1210_3225Metric, symbol Device:C_Small
- added C30: 100n, Capacitor_SMD:C_0805_2012Metric, symbol Device:C_Small
- added C31: 220u, Capacitor_Tantalum_SMD:CP_EIA-7360-38_Kemet-E, symbol Device:C_Polarized_Small_US
- added D5: MBR0530, Diode_SMD:D_SOD-123, symbol Diode:MBR0530
- added J1: SWD, Connector_PinHeader_2.54mm:PinHeader_1x04_P2.54mm_Vertical, symbol Connector_Generic:Conn_01x04
- added J2: USB_C, Connector_USB:USB_C_Receptacle_HRO_TYPE-C-31-M-17, symbol Connector:USB_C_Receptacle_PowerOnly_6P
- added J3: Conn_01x10, Connector_PinHeader_2.54mm:PinHeader_1x10_P2.54mm_Vertical, symbol Connector_Generic:Conn_01x10
- added J4: Conn_01x06, Connector_PinHeader_2.54mm:PinHeader_1x06_P2.54mm_Vertical, symbol Connector_Generic:Conn_01x08
- added L1: 2,2uH, Inductor_SMD:L_APV_APH0650, symbol Device:L
- added L2: 10uH, Inductor_SMD:L_APV_APH0650, symbol Device:L
- added Q3: BC817, Package_TO_SOT_SMD:SOT-23, symbol Transistor_BJT:BC817
- added R61, R62, R63, R64, R65, R69, R72, R76: 10k, Resistor_SMD:R_0603_1608Metric, symbol Device:R_Small
- added R66: 1M, Resistor_SMD:R_0603_1608Metric, symbol Device:R_Small
- added R67, R68: 5k1, Resistor_SMD:R_0603_1608Metric, symbol Device:R_Small
- added R70: 6k8, Resistor_SMD:R_0603_1608Metric, symbol Device:R_Small
- added R71: 1k8, Resistor_SMD:R_0603_1608Metric, symbol Device:R_Small
- added R73: 47k, Resistor_SMD:R_0603_1608Metric, symbol Device:R_Small
- added R74: 330k, Resistor_SMD:R_0603_1608Metric, symbol Device:R_Small
- added R75: 13,3k, Resistor_SMD:R_0603_1608Metric, symbol Device:R_Small
- added RESET: SW_SPST, Button_Switch_SMD:SW_SPST_CK_RS282G05A3, symbol Switch:SW_SPST
- added SW1: RotaryEncoder_Switch_MP, Rotary_Encoder:RotaryEncoder_Alps_EC12E-Switch_Vertical_H20mm, symbol Device:RotaryEncoder_Switch_MP
- added U15: STM32F103C8T6, Package_QFP:LQFP-48_7x7mm_P0.5mm, symbol MCU_ST_STM32F1:STM32F103C8Tx
- added U16: LP2985-3.3, Package_TO_SOT_SMD:SOT-23-5, symbol Regulator_Linear:LP2985-3.3
- added U17: DS1302Z+, Package_SO:SOIC-8_5.3x5.3mm_P1.27mm, symbol Timer_RTC:DS1302Z+
- added U18: MP2307, Package_SO:SOIC-8_3.9x4.9mm_P1.27mm, symbol Regulator_Switching:MP2303ADN
- added U19: LM2733XMF, Package_TO_SOT_SMD:SOT-23-5, symbol Regulator_Switching:LM2733XMF
- added U20: 4017, Package_SO:SOIC-16_3.9x9.9mm_P1.27mm, symbol 4xxx_IEEE:4017
- added Y1: 8MHz, Crystal:Crystal_SMD_HC49-SD, symbol Device:Crystal
- added Y2: 32,768kHz, Crystal:Crystal_AT310_D3.0mm_L10.0mm_Horizontal, symbol Device:Crystal
- R55, R56, R57, R58: value 470 -> 4k7
- R59: value 25k -> 18k
- R60: value 0R -> 10k; footprint Resistor_SMD:R_1206_3216Metric -> Resistor_SMD:R_0603_1608Metric
Connections:
- net +1V2: now also C26.1, L1.2, R71.2
- net +36V: now also C27.1, C29.1, D5.1 (K), R74.2
- net +5V: now also BZ1.1 (+), C20.1, C23.1, C24.1, C28.1, C30.2, C31.1, J2.A9 (VBUS), J2.B9 (VBUS), J4.1 (Pin_1), L2.1, R69.1, R73.1, U16.1 (VIN), U16.3 (ON/~{OFF}), U18.2 (IN), U19.5 (VIN), U20.16 (VDD)
- net COLON: now also U15.15 (PA5)
- net DA: now also U15.10 (PA0)
- net DB: now also U15.11 (PA1)
- net DC: now also U15.12 (PA2)
- net DCLOCK: now also U15.14 (PA4), U20.14 (CP0)
- net DD: now also U15.13 (PA3)
- net DIMPWM: now also U15.46 (PB9)
- net GND: now also BT1.2 (-), C1.2, C10.2, C11.2, C12.2, C13.2, C14.2, C15.2, C16.1, C17.1, C18.2, C19.2, C20.2, C21.2, C22.2, C23.2, C24.2, C26.2, C28.2, C29.2, C30.1, C31.2, C9.1, J1.1 (Pin_1), J2.A12 (GND), J2.B12 (GND), J2.SH (SHIELD), J3.1 (Pin_1), J4.8 (Pin_8), Q3.2 (E), R65.2, R67.2, R68.2, R72.2, R75.2, R76.1, RESET.1 (A), SW1.C, SW1.S2, U15.23 (VSS), U15.35 (VSS), U15.47 (VSS), U15.8 (VSSA), U16.2 (GND), U17.4 (GND), U18.4 (GND), U19.2 (GND), U20.13 (~{CP1}), U20.8 (VSS)
- net RESET: now also U15.16 (PA6), U20.15 (MR)
- net at U4.12 (O7): now also VFD2.5 (e)
- net at U4.13 (O6): now also VFD2.6 (d)
- net at U4.14 (O5): now also VFD2.10 (c)
- net at U4.15 (O4): now also VFD2.1 (b)
- net at U4.16 (O3): now also VFD2.2 (a)
- net at U4.17 (O2): now also VFD2.3 (g)
- net at U4.18 (O1): now also VFD2.4 (f)
- net at U10.12 (O7): now also VFD5.5 (e)
- net at U2.12 (O7): now also VFD1.5 (e)
- net at U2.13 (O6): now also VFD1.6 (d)
- net at U2.14 (O5): now also VFD1.10 (c)
- net at U2.15 (O4): now also VFD1.1 (b)
- net at U2.16 (O3): now also VFD1.2 (a)
- net at U2.17 (O2): now also VFD1.3 (g)
- net at U2.18 (O1): now also VFD1.4 (f)
- net at U8.13 (O6): now also VFD4.6 (d)
- net at U14.13: now also U20.1 (Q5)
- net at U14.11: now also U20.10 (Q4)
- net at U14.3: now also U20.2 (Q1)
- net at U14.1: now also U20.3 (Q0)
- net at U14.5: now also U20.4 (Q2)
- net at U14.9: now also U20.7 (Q3)
- net at U6.18 (O1): now also VFD3.4 (f)
- net at U8.12 (O7): now also VFD4.5 (e)
- net at U8.14 (O5): now also VFD4.10 (c)
- net at U8.15 (O4): now also VFD4.1 (b)
- net at U8.16 (O3): now also VFD4.2 (a)
- net at U8.17 (O2): now also VFD4.3 (g)
- net at U8.18 (O1): now also VFD4.4 (f)
- net +3V3: now reaches R60.1
- net +3V3: now also C12.1, C13.1, C14.1, C15.1, C19.1, J1.4 (Pin_4), R61.1, R62.1, R64.1, U15.1 (VBAT), U15.24 (VDD), U15.36 (VDD), U15.48 (VDD), U15.9 (VDDA), U16.5 (VOUT), U17.1 (VCC2)
- net ENCA: now reaches R60.2
- net ENCA: now also C1.1, SW1.A, U15.25 (PB12)
- net at U6.16 (O3): now also VFD3.2 (a)
- net at U12.14 (O5): now also VFD6.10 (c)
- net at U12.18 (O1): now also VFD6.4 (f)
- net at U6.14 (O5): now also VFD3.10 (c)
- net at U6.13 (O6): now also VFD3.6 (d)
- net at U12.16 (O3): now also VFD6.2 (a)
- net at Q2.1 (B), R59.2: now also R76.2
- net at U6.15 (O4): now also VFD3.1 (b)
- net at U12.12 (O7): now also VFD6.5 (e)
- net at U6.12 (O7): now also VFD3.5 (e)
- net at U6.17 (O2): now also VFD3.3 (g)
- net at VFD5.1 (b): now also U10.15 (O4)
- net at VFD5.10 (c): now also U10.14 (O5)
- net at VFD5.2 (a): now also U10.16 (O3)
- net at VFD5.3 (g): now also U10.17 (O2)
- net at VFD5.4 (f): now also U10.18 (O1)
- net at VFD5.6 (d): now also U10.13 (O6)
- net at VFD6.1 (b): now also U12.15 (O4)
- net at VFD6.3 (g): now also U12.17 (O2)
- net at VFD6.6 (d): now also U12.13 (O6)
- new net: BZ1.2 (-), Q3.3 (C)
- new net: R71.1, R72.1, U18.5 (FB)
- new net: C27.2, R74.1, R75.1, U19.3 (FB)
- new net: J2.A5 (CC1), R68.1
- new net: Q3.1 (B), R63.2
- new net: BT1.1 (+), U17.8 (VCC1)
- new net: C11.1, R64.2, RESET.2 (B), U15.7 (NRST)
- new net: J2.B5 (CC2), R67.1
- new net: R73.2, U19.4 (EN)
- new net: C22.1, R70.2
- new net: C21.1, U18.8 (SS)
- new net: R65.1, U15.44 (BOOT0)
- new net: C18.1, U16.4 (BP)
- new net: U17.2 (X1), Y2.1
- new net: U17.3 (X2), Y2.2
- new net: D5.2 (A), L2.2, U19.1 (SW)
- new net: C25.1, U18.1 (BS)
- new net: C25.2, L1.1, U18.3 (SW)
- new net: R70.1, U18.6 (COMP)
- new net: R69.2, U18.7 (EN)
- new net BUZZER: R63.1, U15.29 (PA8)
- new net ENCB: C9.2, R61.2, SW1.B, U15.26 (PB13)
- new net ENCBUT: C10.1, R62.2, SW1.S1, U15.22 (PB11)
- new net OSC_IN: C17.2, R66.1, U15.5 (PD0), Y1.2
- new net OSC_OUT: C16.2, R66.2, U15.6 (PD1), Y1.1
- new net PA10: J4.4 (Pin_4), U15.31 (PA10)
- new net PA11: J4.5 (Pin_5), U15.32 (PA11)
- new net PA12: J4.6 (Pin_6), U15.33 (PA12)
- new net PA15: J4.7 (Pin_7), U15.38 (PA15)
- new net PA7: J4.2 (Pin_2), U15.17 (PA7)
- new net PA9: J4.3 (Pin_3), U15.30 (PA9)
- new net PB14: J3.9 (Pin_9), U15.27 (PB14)
- new net PB15: J3.10 (Pin_10), U15.28 (PB15)
- new net PB2: J3.2 (Pin_2), U15.20 (PB2)
- new net PB3: J3.3 (Pin_3), U15.39 (PB3)
- new net PB4: J3.4 (Pin_4), U15.40 (PB4)
- new net PB5: J3.5 (Pin_5), U15.41 (PB5)
- new net PB6: J3.6 (Pin_6), U15.42 (PB6)
- new net PB7: J3.7 (Pin_7), U15.43 (PB7)
- new net PB8: J3.8 (Pin_8), U15.45 (PB8)
- new net RTC_CLK: U15.21 (PB10), U17.7 (SCLK)
- new net RTC_DAT: U15.19 (PB1), U17.6 (I/O)
- new net RTC_RES: U15.18 (PB0), U17.5 (CE)
- new net SWCLK: J1.2 (Pin_2), U15.37 (PA14)
- new net SWDIO: J1.3 (Pin_3), U15.34 (PA13)
- no-connect marks 17 -> 18
Other:
- note added: "5v-1,2v Power supply"
- note added: "5v-30v Power supply"
- note added: "5v-3v3 Power supply"
- note added: "Buzzer"
- note added: "Dallas RTC"
- note added: "MCU"
- note added: "Rotary Encoder"
- note added: "VFD CONTROL"
- note removed: "1206 Jumper"
- note removed: "Power supply"
- moved on the sheet: C2, C3, C4, C5, C6, C7, C8, D1, D2, D3, D4, Q2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

Commit message: New board draft
Parts:
- added H1, H2, H3, H4: MountingHole, MountingHole:MountingHole_2.7mm_M2.5_DIN965_Pad, symbol Mechanical:MountingHole
- D1, D2, D3, D4: footprint LED_THT:LED_D3.0mm_Clear -> LED_SMD:LED_0603_1608Metric
- J4: footprint Connector_PinHeader_2.54mm:PinHeader_1x06_P2.54mm_Vertical -> Connector_PinHeader_2.54mm:PinHeader_1x08_P2.54mm_Vertical
- VFD1, VFD2, VFD3, VFD4, VFD5, VFD6: footprint Library:IV-6 -> Library:IV-6_Horizontal
- renumbered RESET to RESET1

Commit message: New 4-layer board layout
Parts:
- removed BZ1: Buzzer, Buzzer_Beeper:Buzzer_12x9.5RM7.6, symbol Device:Buzzer
- removed Y2: 32,768kHz, Crystal:Crystal_AT310_D3.0mm_L10.0mm_Horizontal, symbol Device:Crystal
- added BZ1: (no value), Library:HCT5020, symbol CustomLibrary:HCT5020
- added Y2: 32.768 KHz, Crystal:Crystal_SMD_SeikoEpson_MC306-4Pin_8.0x3.2mm, symbol Device:Crystal_GND23
- Y1: footprint Crystal:Crystal_SMD_HC49-SD -> Crystal:Crystal_SMD_5032-2Pin_5.0x3.2mm_HandSoldering
Connections:
- net +3V3: now also BZ1.1 (+)
- net DCLOCK: now also U15.17 (PA7); no longer U15.14 (PA4)
- net at Q3.3 (C): now also BZ1.2 (-)
- net at U17.2 (X1): now also Y2.4
- net at U17.3 (X2): now also Y2.1
- net PA7 renamed PA4
- net PA4: now also U15.14 (PA4); no longer U15.17 (PA7)
- new net: Y2.2 (G), Y2.3 (G)
- no-connect marks 18 -> 20

Commit message: Updated schematics pdf
Parts:
- added TP1: 3V3, TestPoint:TestPoint_Pad_1.0x1.0mm, symbol Connector:TestPoint_Alt
- added TP2: 5V, TestPoint:TestPoint_Pad_1.0x1.0mm, symbol Connector:TestPoint_Alt
- added TP3: 1V2, TestPoint:TestPoint_Pad_1.0x1.0mm, symbol Connector:TestPoint_Alt
- added TP4: 30v, TestPoint:TestPoint_Pad_1.0x1.0mm, symbol Connector:TestPoint_Alt
Connections:
- net +1V2: now also TP3.1
- net +36V: now also TP4.1
- net +3V3: now also TP1.1
- net +5V: now also TP2.1
Other:
- note added: "2026"
- note added: "A.Nerovny"
- note added: "github.com/nerovny/IV-6-VFD-Clock"
- note added: "ИВ-6 VFD Digital Clock"
- moved on the sheet: H1, H2, H3, H4

Commit message: Updated schematic and board
Parts:
- added C19: 100n, Capacitor_SMD:C_0603_1608Metric, symbol Device:C_Small
- added F1: 0,75A 6V, Fuse:Fuse_1210_3225Metric, symbol Device:Fuse
- added J3: Power, Connector_JST:JST_XH_B2B-XH-A_1x02_P2.50mm_Vertical, symbol Connector_Generic:Conn_01x02
- added R21: 10k, Resistor_SMD:R_0603_1608Metric, symbol Device:R_Small
- added R24: 0, Resistor_SMD:R_0603_1608Metric, symbol Device:R_Small
- added SW2: MODE, Button_Switch_THT:SW_Tactile_SPST_Angled_PTS645Vx39-2LFS, symbol Switch:SW_SPST
- renumbered C20 to C1, C19 to C10, C22 to C11, C25 to C12, C27 to C13, C29 to C14, C26 to C15, C11 to C16, C16 to C18, C1 to C2, C31 to C20, C12 to C21, C13 to C22, C30 to C23, C14 to C24, C15 to C25, C8 to C26, C2 to C27, C3 to C28, C4 to C29, C9 to C3, C5 to C30, C6 to C31, C7 to C32, C24 to C4, C23 to C5, C18 to C6, C21 to C7, C10 to C8, C28 to C9, D5 to D1, D1 to D2, D2 to D3, D3 to D4, D4 to D5, J2 to J1, J1 to J2, J3 to J4, J4 to J5, L2 to L1, L1 to L2, Q3 to Q1, R61 to R1, R72 to R10, R71 to R11, R55 to R12, R59 to R13, R76 to R14, R56 to R15, R57 to R16, R58 to R17, R64 to R18, R65 to R19, R60 to R2, R66 to R20, R67 to R22, R68 to R23, R9 to R25, R10 to R26, R19 to R27, R37 to R29, R62 to R3, R46 to R30, R1 to R31, R18 to R32, R27 to R33, R36 to R34, R45 to R35, R54 to R36, R69 to R4, R73 to R5, R70 to R6, R75 to R7, R63 to R8, R74 to R9, TP2 to TP1, TP1 to TP2, TP4 to TP3, TP3 to TP4, U16 to U1, U5 to U10, U7 to U11, U9 to U12, U11 to U13, U2 to U14, U4 to U15, U6 to U16, U8 to U17, U10 to U18, U12 to U19, U18 to U2, U19 to U3, U17 to U4, U15 to U5, U14 to U6, U20 to U7, U1 to U8, U3 to U9, Y2 to Y1, Y1 to Y2
Connections:
- net +3V3: now also R21.1
- net +5V: now also F1.1, J3.2 (Pin_2); no longer J1.A9 (VBUS), J1.B9 (VBUS)
- net GND: now also C19.2, J3.1 (Pin_1), SW2.1 (A)
- net PB15: now also R24.2
- new net: C19.1, R21.2, R24.1, SW2.2 (B)
- new net: F1.2, J1.A9 (VBUS), J1.B9 (VBUS)
Other:
- moved on the sheet: C20, J2, J4, J5

Commit message: Replaced the RTC chip with PCF8563T
Parts:
- removed U4: DS1302Z+, Package_SO:SOIC-8_5.3x5.3mm_P1.27mm, symbol Timer_RTC:DS1302Z+
- added C33: 100n, Capacitor_SMD:C_0603_1608Metric, symbol Device:C_Small
- added C34: 22p, Capacitor_SMD:C_0402_1005Metric, symbol Device:C_Small
- added D7: BAV70, Package_TO_SOT_SMD:SOT-23, symbol Diode:BAV70
- added R37, R38, R39: 4k7, Resistor_SMD:R_0402_1005Metric, symbol Device:R_Small
- added TP5: CLKO, TestPoint:TestPoint_Pad_1.0x1.0mm, symbol Connector:TestPoint_Alt
- added U20: PCF8563T, Package_SO:SOIC-8_3.9x4.9mm_P1.27mm, symbol Timer_RTC:PCF8563T
Connections:
- net +3V3: now also D7.1 (A), R37.1, R38.1, R39.1
- net GND: now also C33.1, C34.2, U20.4 (VSS)
- net RTC_CLK: now also R37.2, U20.6 (SCL)
- net RTC_DAT: now also R38.2, U20.5 (SDA)
- net at BT1.1 (+): now also D7.2 (A)
- net at Y1.4: now also C34.1, U20.1 (OSCI)
- net at Y1.1: now also U20.2 (OSCO)
- net RTC_RES renamed RTC_INT
- net RTC_INT: now also R39.2, U20.3 (~{INT})
- new net: TP5.1, U20.7 (CLKO)
- new net: C33.2, D7.3 (K), U20.8 (VDD)
Other:
- note added: "RTC"
- note removed: "Dallas RTC"
- moved on the sheet: BT1, Y1
